File: eagle/log-controller-v2.brd (EAGLE design)
At the start: 63.2 x 80 mm, 23 parts, among them Q1 IRLB8721PBFTO220AB, T1 2N3055, T2 BC547, X1 Power/Motor

Commit message: Changed a resistor due to the electronic gearbox not working.
Seems not to have solved it completely... back to the drawing board.
Parts:
- R5: value 1K -> 330
Changed lines of the file:
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@@
 <attribute name="MF" value="VISHAY/TELEFUNKEN" x="12.7" y="62.23" size="1.778" layer="27" rot="R180" display="off"/>
 </element>
-<element name="R5" library="resistor" package="0207/12" value="1K" x="30.48" y="62.23" rot="R180"/>
+<element name="R5" library="resistor" package="0207/12" value="330" x="30.48" y="62.23" rot="R180"/>
 <element name="R6" library="resistor" package="0207/12" value="10K" x="15.24" y="29.21"/>
 <element name="R7" library="resistor" package="0207/12" value="10K" x="30.48" y="66.04" rot="R180"/>
